File: PCB/pcb-wiring-plan/pcb-wiring-plan.kicad_sch (KiCad schematic)
At the start: 19 parts, among them J1 Pinout, J12 Conn_01x02_Pin, J13 XH6, J14 Conn_01x12_Socket, J15 Conn_01x04_Socket, J16 Conn_01x08_Socket, J18 XH6, J2 XH6, J3 XH6, J4 Pinout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

Commit message: wiring plan updates
Parts:
- removed J12, J9: Conn_01x02_Pin, symbol Connector:Conn_01x02_Pin
- removed J15: Conn_01x04_Socket, symbol Connector:Conn_01x04_Socket
- added J9: XH6, symbol Connector:Conn_01x06_Socket
Other:
- note added: "VLP2"
- note removed: "XH2"
- note removed: "XH2*"
- note removed: "XH4"
