File: PCB/power_splitter/power_splitter.kicad_pcb (KiCad board)
At the start: 2 copper layers, 93 x 69 mm, 29 parts, among them J1 B02P-VL, J2 B02P-VL, J3 B02P-VL, J4 PJ-082BH, Q2 IRLZ44N, U1 AP62300TWU, U2 AP62300TWU

Commit message: power stuff
Parts:
- moved L2 39.2 mm to (124.4, 49.5), turned to 0 degrees
- moved L1 27.0 mm to (103.0, 59.5), turned to -90 degrees
- moved R1 26.3 mm to (86.0, 71.3), turned to 90 degrees
- moved C5 21.4 mm to (86.5, 76.5)
- moved C6 21.4 mm to (92.5, 76.5)
- moved C2 17.9 mm to (97.5, 53.0)
- moved C4 15.0 mm to (80.5, 65.0), turned to 90 degrees
- moved F1 14.4 mm to (99.0, 44.8), turned to -90 degrees
- moved J2 11.3 mm to (109.4, 82.4)
- moved J3 11.3 mm to (124.2, 82.5)
- moved J4 9.94 mm to (83.5, 41.1), turned to -90 degrees
- moved C3 9.72 mm to (97.0, 67.0)
- moved U2 9.65 mm to (96.4, 60.5)
- moved R7 8.89 mm to (145.0, 37.3)
- moved R8 8.87 mm to (149.5, 37.2), turned to -90 degrees
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Connections:
- net Net-(C10-Pad1) renamed 3V_Line
- net Vout renamed 5V_Line
- J4 pad SH1: unconnected-(J4-SHIELD-PadSH1) -> GND
- J4 pad SH2: unconnected-(J4-SHIELD__1-PadSH2) -> GND
- J4 pad SH3: unconnected-(J4-SHIELD__2-PadSH3) -> GND
- J4 pad SH4: unconnected-(J4-SHIELD__3-PadSH4) -> GND
Routing:
- net 5V_Line: track 0.00 -> 76.6 mm
- net 3V_Line: track 0.00 -> 48.0 mm
- net /electronics branch: track 0.00 -> 40.6 mm
- net GND: track 35.3 -> 67.3 mm, vias 14 -> 16
- net Net-(U1-FB): track 0.00 -> 20.9 mm
- net Net-(U2-EN): track 0.00 -> 16.7 mm
- net Net-(U2-FB): track 0.00 -> 16.4 mm
- net Net-(U2-SW): track 0.00 -> 15.3 mm
- net Net-(Q2-G): track 0.00 -> 12.1 mm
- net Net-(U1-SW): track 0.00 -> 11.7 mm
- net Net-(F3-Pad2): track 0.00 -> 9.77 mm
- net Net-(Q2-D): track 0.00 -> 8.52 mm
- net Net-(U1-BST): track 0.00 -> 6.73 mm
- net Net-(U2-BST): track 0.00 -> 5.92 mm
- net (no net): vias 1 -> 0
Other:
- board size 93 x 69 mm -> 88 x 62 mm
