File: PCB/main_pcb/main_pcb/main_pcb.kicad_sch (KiCad schematic)
At the start: 16 parts, among them J1 Conn_01x20_Socket, J2 Conn_01x20_Socket, J3 B02P-VL, J4 B02P-VL, J5 B8B-XH-A, J6 B8B-XH-A, J7 B8B-XH-A, J8 B8B-XH-A, U1 MCP3208, U2 MCP3208, U3 APDS-9006-020

Commit message: Added switch board connector and display board connector circuitry to main pcb.
Parts:
- added C10, C2, C3, C4, C5, C6, C7, C8, C9: C1206C101K1HACTU, CAPC340180_88N_KEM, symbol C1206C101K1HACTU:C1206C101K1HACTU
- added J10, J12, J9: B6B-XH-A, Connector_JST:JST_XH_B6B-XH-A_1x06_P2.50mm_Vertical, symbol B6B-XH-A:B6B-XH-A
- added J11: B8B-XH-A, Connector_JST:JST_XH_B8B-XH-A_1x08_P2.50mm_Vertical, symbol B8B-XH-A:B8B-XH-A
- added R10, R2, R3, R4, R5, R6, R7, R8, R9: 8.25k, YAG_MF25_YAG, symbol ul_MFP-25BRD52-10K:MFP-25BRD52-10K
- added U10, U11, U12, U4, U5, U6, U7, U8, U9: APDS-9006-020, APDS-9006-020:XDCR_APDS-9006-020, symbol APDS-9006-020:APDS-9006-020
Connections:
- net +3.3V: now also J10.1, J11.1, J9.1, U10.2 (VCC), U10.3 (VCC__1), U11.2 (VCC), U11.3 (VCC__1), U12.2 (VCC), U12.3 (VCC__1), U4.2 (VCC), U4.3 (VCC__1), U5.2 (VCC), U5.3 (VCC__1), U6.2 (VCC), U6.3 (VCC__1), U7.2 (VCC), U7.3 (VCC__1), U8.2 (VCC), U8.3 (VCC__1), U9.2 (VCC), U9.3 (VCC__1)
- net BTN0: now also J12.2
- net BTN1: now also J12.3
- net BTN2: now also J12.4
- net BTN3: now also J12.5
- net DISP REGSEL: now also J11.7
- net DISP_RST: now also J11.6
- net GND: now also J10.2, J10.4, J11.2, J11.4, J12.1, J12.6, J9.2, J9.4
- net OpIn1: now also C2.1, R2.1, U4.1 (OUT)
- net OpIn2: now also C3.1, R3.1, U5.1 (OUT)
- net OpIn3: now also C4.1, R4.1, U6.1 (OUT)
- net OpIn4: now also C5.1, R5.1, U7.1 (OUT)
- net OpIn5: now also C6.1, R6.1, U8.1 (OUT)
- net OpIn6: now also C7.1, R7.1, U9.1 (OUT)
- net OpIn7: now also C8.1, R8.1, U10.1 (OUT)
- net OpIn8: now also C9.1, R9.1, U11.1 (OUT)
- net OpIn9: now also C10.1, R10.1, U12.1 (OUT)
- net OpOut1: now also C2.2, R2.2
- net OpOut2: now also C3.2, R3.2
- net OpOut3: now also C4.2, R4.2
- net OpOut4: now also C5.2, R5.2
- net OpOut5: now also C6.2, R6.2
- net OpOut6: now also C7.2, R7.2
- net OpOut7: now also C8.2, R8.2
- net OpOut8: now also C9.2, R9.2
- net OpOut9: now also C10.2, R10.2
- net SPI0_CSn: now also J11.8
- net SPI0_SCK: now also J11.3
- net SPI0_TX: now also J11.5
- net QH1: now reaches J2.10 (Pin_10)
- net QH1: now also J9.6
- net SH1: now reaches J2.7 (Pin_7)
- net SH1: now also J9.3
- net CLK: now reaches J2.9 (Pin_9)
- net CLK: now also J10.5, J9.5
- net SH2: now reaches J1.1 (Pin_1)
- net SH2: now also J10.3
- net QH2: now reaches J1.2 (Pin_2)
- net QH2: now also J10.6
- no-connect marks 26 -> 21
Other:
- note added: "Fan Connectors"
- moved on the sheet: J5, J6, J7, J8

Commit message: Finished circuit layout for the main PCB exlcuding the fan headers.
Parts:
- removed C10: C1206C101K1HACTU, CAPC340180_88N_KEM, symbol C1206C101K1HACTU:C1206C101K1HACTU
- removed R10: 8.25k, YAG_MF25_YAG, symbol ul_MFP-25BRD52-10K:MFP-25BRD52-10K
- added C1: 100p, C1206C101K1HACTU:CAPC340180_88N_KEM, symbol C1206C101K1HACTU:C1206C101K1HACTU
- added R1: 8.25k, ul_MFP-25BRD52-10K:YAG_MF25_YAG, symbol ul_MFP-25BRD52-10K:MFP-25BRD52-10K
- C0: renamed from C1; value C1206C101K1HACTU -> 100p; footprint CAPC340180_88N_KEM -> C1206C101K1HACTU:CAPC340180_88N_KEM
- C2, C3, C4, C5, C6, C7, C8, C9: value C1206C101K1HACTU -> 100p; footprint CAPC340180_88N_KEM -> C1206C101K1HACTU:CAPC340180_88N_KEM
- J5, J6, J7, J8: footprint B8B-XH-A:JST_B8B-XH-A -> B8B_XH_A:JST_B8B-XH-A
- OpAmp1, OpAmp2, OpAmp3: footprint LMC660CM:SOIC127P600X175-14N -> LMC660CMX_NOPB:SOIC127P600X175-14N
- R0: renamed from R1; footprint YAG_MF25_YAG -> ul_MFP-25BRD52-10K:YAG_MF25_YAG
- R2, R3, R4, R5, R6, R7, R8, R9: footprint YAG_MF25_YAG -> ul_MFP-25BRD52-10K:YAG_MF25_YAG
- U1, U2: footprint (none) -> MCP3208_CI_P:DIP254P762X432-16
- U10, U11, U12, U3, U4, U5, U6, U7, U8, U9: footprint APDS-9006-020:XDCR_APDS-9006-020 -> APDS_9006_020:XDCR_APDS-9006-020
Connections:
- net +5V: now also OpAmp2.4 (V+)
- net OpIn1: now also C1.1, R1.1; no longer C2.1, R2.1
- net OpIn2: now also C2.1, R2.1; no longer C3.1, R3.1
- net OpIn3: now also C3.1, R3.1; no longer C4.1, R4.1
- net OpIn4: now also C4.1, R4.1; no longer C5.1, R5.1
- net OpIn5: now also C5.1, R5.1; no longer C6.1, R6.1
- net OpIn6: now also C6.1, R6.1; no longer C7.1, R7.1
- net OpIn7: now also C7.1, R7.1; no longer C8.1, R8.1
- net OpIn8: now also C8.1, R8.1; no longer C9.1, R9.1
- net OpIn9: now also C9.1, R9.1
- net OpOut1: now also C1.2, R1.2; no longer C2.2, R2.2
- net OpOut2: now also C2.2, R2.2; no longer C3.2, R3.2
- net OpOut3: now also C3.2, R3.2; no longer C4.2, R4.2
- net OpOut4: now also C4.2, R4.2; no longer C5.2, R5.2
- net OpOut5: now also C5.2, R5.2; no longer C6.2, R6.2
- net OpOut6: now also C6.2, R6.2; no longer C7.2, R7.2
- net OpOut7: now also C7.2, R7.2; no longer C8.2, R8.2
- net OpOut8: now also C8.2, R8.2; no longer C9.2, R9.2
- net OpOut9: now also C9.2, R9.2
- no-connect marks 21 -> 23
Other:
- moved on the sheet: C0, OpAmp1, R0, U3

Commit message: Added pi 1x20 pin socket for now (subject to change).
Parts:
- J1, J2: footprint (none) -> Connector_PinSocket_1.00mm:PinSocket_1x20_P1.00mm_Vertical
Changed lines of the file:
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@@
 	)
 	(symbol
-		(lib_id "Connector:Conn_01x20_Socket")
-		(at 325.12 41.91 0)
-		(mirror y)
-		(unit 1)
-		(exclude_from_sim no)
-		(in_bom yes)
-		(on_board yes)
-		(dnp no)
-		(property "Reference" "J2"
-			(at 325.12 15.494 0)
-			(effects
-				(font
-					(size 1.27 1.27)
-				)
-			)
-		)
-		(property "Value" "Conn_01x20_Socket"
-			(at 325.755 69.85 0)
-			(effects
-				(font
-					(size 1.27 1.27)
-				)
-				(hide yes)
-			)
-		)
-		(property "Footprint" ""
-			(at 325.12 41.91 0)
-			(effects
-				(font
-					(size 1.27 1.27)
-				)
-				(hide yes)
-			)
-		)
-		(property "Datasheet" "~"
-			(at 325.12 41.91 0)
-			(effects
-				(font
-					(size 1.27 1.27)
-				)
-				(hide yes)
-			)
-		)
-		(property "Description" "Generic connector, single row, 01x20, script generated"
-			(at 325.12 41.91 0)
-			(effects
-				(font
-					(size 1.27 1.27)
-				)
-				(hide yes)
-			)
-		)
-		(pin "9"
-		)
-		(pin "12"
-		)
-		(pin "6"
-		)
-		(pin "16"
-		)
-		(pin "17"
-		)
-		(pin "1"
-		)
-		(pin "11"
-		)
-		(pin "13"
-		)
-		(pin "3"
-		)
-		(pin "4"
-		)
-		(pin "2"
-		)
-		(pin "5"
-		)
-		(pin "7"
-		)
-		(pin "8"
-		)
-		(pin "10"
-		)
-		(pin "14"
-		)
-		(pin "15"
-		)
-		(pin "20"
-		)
-		(pin "18"
-		)
-		(pin "19"
-		)
-		(instances
-			(project "main_pcb"
-				(path "/9e1b86fa-37cc-48d2-968d-4a7578d4873f"
-					(reference "J2")
-					(unit 1)
-				)
-			)
-		)
-	)
-	(symbol
 		(lib_id "power:+3V3")
 		(at 109.22 132.08 270)
@@
 			)
 		)
-		(property "Footprint" ""
+		(property "Footprint" "Connector_PinSocket_1.00mm:PinSocket_1x20_P1.00mm_Vertical"
 			(at 299.72 41.91 0)
 			(effects
@@
 					(unit 1)
 				)
+			)
+		)
+	)
+	(symbol
+		(lib_id "Connector:Conn_01x20_Socket")
+		(at 325.12 41.91 0)
+		(mirror y)
+		(unit 1)
+		(exclude_from_sim no)
+		(in_bom yes)
+		(on_board yes)
+		(dnp no)
+		(property "Reference" "J2"
+			(at 325.12 15.494 0)
+			(effects
+				(font
+					(size 1.27 1.27)
+				)
+			)
+		)
+		(property "Value" "Conn_01x20_Socket"
+			(at 323.85 44.4499 0)
+			(effects
+				(font
+					(size 1.27 1.27)
+				)
+				(justify left)
+				(hide yes)
+			)
+		)
+		(property "Footprint" "Connector_PinSocket_1.00mm:PinSocket_1x20_P1.00mm_Vertical"
+			(at 325.12 41.91 0)
+			(effects
+				(font
+					(size 1.27 1.27)
+				)
+				(hide yes)
+			)
+		)
+		(property "Datasheet" "~"
+			(at 325.12 41.91 0)
+			(effects
+				(font
+					(size 1.27 1.27)
+				)
+				(hide yes)
+			)
+		)
+		(property "Description" "Generic connector, single row, 01x20, script generated"
+			(at 325.12 41.91 0)
+			(effects
+				(font
+					(size 1.27 1.27)
+				)
+				(hide yes)
+			)
+		)
+		(pin "1"
+		)
+		(pin "2"
+		)
+		(pin "3"
+		)
+		(pin "4"
+		)
+		(pin "5"
+		)
+		(pin "6"
+		)
+		(pin "7"
+		)
+		(pin "8"
+		)
+		(pin "11"
+		)
+		(pin "14"
+		)
+		(pin "10"
+		)
+		(pin "18"
+		)
+		(pin "12"
+		)
+		(pin "9"
+		)
+		(pin "20"
+		)
+		(pin "17"
+		)
+		(pin "16"
+		)
+		(pin "15"
+		)
+		(pin "19"
+		)
+		(pin "13"
+		)
+		(instances
+			(project "main_pcb"
+				(path "/9e1b86fa-37cc-48d2-968d-4a7578d4873f"
+					(reference "J2")
+					(unit 1)
+				)

Commit message: Added fan and sd card header among other things to the main pcb.
Parts:
- added J13, J14: B8B-XH-A, Connector_JST:JST_XH_B8B-XH-A_1x08_P2.50mm_Vertical, symbol B8B-XH-A:B8B-XH-A
Connections:
- net +3.3V: now also J13.1
- net +5V: now also J14.2, J14.4
- net GND: now also J13.2, J14.1, J14.3; no longer J10.4, J9.4
- net SPI1_RX: now also J10.6, J9.6, J13.5
- net SPI1_SCK: now also J10.5, J9.5, J13.3
- net SPI1_TX: now also J10.3, J9.3, J13.4
- removed net CLK: J10.5, J2.9 (Pin_9), J9.5
- net GPIO6: no longer names the net of J1.9 (Pin_9)
- net QH1 renamed SPI1_CSn_TD1
- net SPI1_CSn_TD1: now also J10.4; no longer J9.6
- net QH2 renamed SPI1_CDn_SD
- net SPI1_CDn_SD: now also J13.7; no longer J10.6
- net RUN: no longer names the net of J2.11 (Pin_11)
- net SH1: no longer names the net of J2.7 (Pin_7)
- net SH1: no longer J9.3
- net SH2 renamed SPI1_CSn_SD
- net SPI1_CSn_SD: now also J13.6; no longer J10.3
- new net SPI1_CSn_TD0: J2.9 (Pin_9), J9.4
- no-connect marks 23 -> 31
Other:
- note added: "BTNs"
- note added: "LCD"
- note added: "SD Card"

Commit message: Started layout of the main PCB. God help me for I have sinned :(
Parts:
- J1, J2: footprint Connector_PinSocket_1.00mm:PinSocket_1x20_P1.00mm_Vertical -> Connector_PinSocket_2.54mm:PinSocket_1x20_P2.54mm_Vertical
- J5, J6, J7, J8: footprint B8B_XH_A:JST_B8B-XH-A -> Connector_JST:JST_XH_B8B-XH-A_1x08_P2.50mm_Vertical
Connections:
- net +3.3V: no longer U4.2 (VCC), U4.3 (VCC__1)
- net GND: now also J13.4, J13.8; no longer J3.2
- net HEATER_ON: now also J3.2
- net OpIn0: now also OpAmp1.10 (IN3+); no longer OpAmp1.3 (IN1+)
- net OpIn1: now also OpAmp1.12 (IN4+), U4.4 (NC); no longer OpAmp1.5 (IN2+), U4.1 (OUT)
- net OpIn2: now also C9.1, OpAmp1.5 (IN2+), R9.1, U12.1 (OUT); no longer C2.1, OpAmp1.10 (IN3+), R2.1, U5.1 (OUT)
- net OpIn3: now also C8.1, OpAmp1.3 (IN1+), R8.1, U11.1 (OUT); no longer C3.1, OpAmp1.12 (IN4+), R3.1, U6.1 (OUT)
- net OpIn4: now also C2.1, R2.1, U5.1 (OUT); no longer C4.1, R4.1, U7.1 (OUT)
- net OpIn5: now also C3.1, R3.1, U6.1 (OUT); no longer C5.1, R5.1, U8.1 (OUT)
- net OpIn6: now also C7.1, OpAmp2.12 (IN4+), R7.1, U10.1 (OUT); no longer C6.1, OpAmp2.10 (IN3+), R6.1, U9.1 (OUT)
- net OpIn7: now also C6.1, OpAmp2.10 (IN3+), R6.1, U9.1 (OUT); no longer C7.1, OpAmp2.12 (IN4+), R7.1, U10.1 (OUT)
- net OpIn8: now also C4.1, R4.1, U7.1 (OUT); no longer C8.1, R8.1, U11.1 (OUT)
- net OpIn9: now also C5.1, OpAmp3.12 (IN4+), R5.1, U8.1 (OUT); no longer C9.1, OpAmp3.5 (IN2+), R9.1, U12.1 (OUT)
- net OpOut0: now also OpAmp1.8 (OUT3), U1.8 (CH7); no longer OpAmp1.1 (OUT1), U2.1 (CH0)
- net OpOut1: now also OpAmp1.14 (OUT4), U1.7 (CH6); no longer OpAmp1.7 (OUT2), U2.2 (CH1)
- net OpOut2: now also C9.2, OpAmp1.7 (OUT2), R9.2, U2.1 (CH0); no longer C2.2, OpAmp1.8 (OUT3), R2.2, U2.3 (CH2)
- net OpOut3: now also C8.2, OpAmp1.1 (OUT1), R8.2, U2.2 (CH1); no longer C3.2, OpAmp1.14 (OUT4), R3.2, U2.4 (CH3)
- net OpOut4: now also C2.2, R2.2, U1.6 (CH5); no longer C4.2, R4.2, U2.5 (CH4)
- net OpOut5: now also C3.2, R3.2, U1.5 (CH4); no longer C5.2, R5.2, U1.1 (CH0)
- net OpOut6: now also C7.2, OpAmp2.14 (OUT4), R7.2, U2.3 (CH2); no longer C6.2, OpAmp2.8 (OUT3), R6.2, U1.2 (CH1)
- net OpOut7: now also C6.2, OpAmp2.8 (OUT3), R6.2, U2.4 (CH3); no longer C7.2, OpAmp2.14 (OUT4), R7.2, U1.3 (CH2)
- net OpOut8: now also C4.2, R4.2; no longer C8.2, R8.2
- net OpOut9: now also C5.2, OpAmp3.14 (OUT4), R5.2, U2.5 (CH4); no longer C9.2, OpAmp3.7 (OUT2), R9.2, U1.5 (CH4)
- net SPI1_CSn_SD: now also J13.7; no longer J13.6
- net SPI1_RX: now also J13.6; no longer J13.5
- net SPI1_TX: now also J13.5; no longer J13.4
- net SPI1_CDn_SD: no longer names the net of J1.2 (Pin_2)
- net SPI1_CDn_SD: no longer J13.7

Commit message: And falling into a place where two layers met, they ran the PCB  aground; and the forepart stuck fast, and remained unmoveable, but the hinder part was broken with the violence of the photodiodes.
Connections:
- net +3.3V: now also U4.2 (VCC), U4.3 (VCC__1)
- net OpIn1: now also U4.1 (OUT); no longer U4.4 (NC)
- net SPI1_CSn_TD0: now also J2.10 (Pin_10), J9.6; no longer J2.9 (Pin_9), J9.4
- net SPI1_CSn_TD1: now also J10.6, J2.9 (Pin_9); no longer J10.4, J2.10 (Pin_10)
- net SPI1_RX: now also J10.3, J9.3; no longer J10.6, J9.6
- net SPI1_SCK: now also J10.4, J13.5, J9.4; no longer J10.5, J13.3, J9.5
- net SPI1_TX: now also J10.5, J13.3, J9.5; no longer J10.3, J13.5, J9.3

Commit message: The PCB is the resurrection and the life; he that believeth in it, though it were dead, yet shall he live.
Parts:
- U10, U11, U12, U3, U4, U5, U6, U7, U8, U9: footprint APDS_9006_020:XDCR_APDS-9006-020 -> APDS_9006_020:photodiode_v3
Changed lines of the file:
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@@
 			)
 		)
-		(property "Footprint" "APDS_9006_020:XDCR_APDS-9006-020"
+		(property "Footprint" "APDS_9006_020:photodiode_v3"
 			(at 160.02 132.08 0)
 			(effects
@@
 			)
 		)
-		(property "Footprint" "APDS_9006_020:XDCR_APDS-9006-020"
+		(property "Footprint" "APDS_9006_020:photodiode_v3"
 			(at 160.02 157.48 0)
 			(effects
@@
 			)
 		)
-		(property "Footprint" "APDS_9006_020:XDCR_APDS-9006-020"
+		(property "Footprint" "APDS_9006_020:photodiode_v3"
 			(at 96.52 132.08 0)
 			(effects
@@
 			)
 		)
-		(property "Footprint" "APDS_9006_020:XDCR_APDS-9006-020"
+		(property "Footprint" "APDS_9006_020:photodiode_v3"
 			(at 160.02 106.68 0)
 			(effects
@@
 			)
 		)
-		(property "Footprint" "APDS_9006_020:XDCR_APDS-9006-020"
+		(property "Footprint" "APDS_9006_020:photodiode_v3"
 			(at 96.52 157.48 0)
 			(effects
@@
 			)
 		)
-		(property "Footprint" "APDS_9006_020:XDCR_APDS-9006-020"
+		(property "Footprint" "APDS_9006_020:photodiode_v3"
 			(at 160.02 208.28 0)
 			(effects
@@
 			)
 		)
-		(property "Footprint" "APDS_9006_020:XDCR_APDS-9006-020"
+		(property "Footprint" "APDS_9006_020:photodiode_v3"
 			(at 96.52 208.28 0)
 			(effects
@@
 			)
 		)
-		(property "Footprint" "APDS_9006_020:XDCR_APDS-9006-020"
+		(property "Footprint" "APDS_9006_020:photodiode_v3"
 			(at 96.52 106.68 0)
 			(effects
@@
 			)
 		)
-		(property "Footprint" "APDS_9006_020:XDCR_APDS-9006-020"
+		(property "Footprint" "APDS_9006_020:photodiode_v3"
 			(at 96.52 182.88 0)
 			(effects
@@
 			)
 		)
-		(property "Footprint" "APDS_9006_020:XDCR_APDS-9006-020"
+		(property "Footprint" "APDS_9006_020:photodiode_v3"
 			(at 160.02 182.88 0)
 			(effects

Commit message: Rejoice always, pray continually, give thanks in all circumstances, for this is the PCB’s will for you.
Parts:
- renumbered U2 to ADC0, U1 to ADC1, J12 to BTN_Header1, J14 to Fan_Header1, J11 to LCD_Header1, U3 to Photo0, U4 to Photo1, U12 to Photo2, U11 to Photo3, U5 to Photo4, U6 to Photo5, U9 to Photo7, U7 to Photo8, U8 to Photo9, J3 to Power_Connector_3V3, J4 to Power_Connector_5V1, J13 to SD_Header1, J9 to SW0_Header1, J10 to SW1_Header1, J8 to Temp0_Header1, J7 to Temp1_Header1, J6 to Temp2_Header1, J5 to Temp3_Header1, U10 to UPhoto6
Connections:
- net +3.3V: now also Temp1_Header1.6, Temp2_Header1.7, Temp3_Header1.6, Temp3_Header1.7
- no-connect marks 31 -> 27
