File: PCB/main_pcb/main_pcb/main_pcb.kicad_sch (KiCad schematic)
At the start: 52 parts, among them J1 Conn_01x20_Socket, J2 Conn_01x20_Socket, J3 Conn_01x09_Socket, Q1 DMG2305UX-7, SW0_Header1 B6B-XH-A, SW1_Header1 B6B-XH-A

Commit message: Updated main PCB
Connections:
- net GND: now also OpAmp1.10 (IN3+), OpAmp1.12 (IN4+), OpAmp1.3 (IN1+), OpAmp1.5 (IN2+), OpAmp2.10 (IN3+), OpAmp2.12 (IN4+), OpAmp2.3 (IN1+), OpAmp2.5 (IN2+), OpAmp3.12 (IN4+), OpAmp3.3 (IN1+); no longer OpAmp1.13 (IN4-), OpAmp1.2 (IN1-), OpAmp1.6 (IN2-), OpAmp1.9 (IN3-), OpAmp2.13 (IN4-), OpAmp2.2 (IN1-), OpAmp2.6 (IN2-), OpAmp2.9 (IN3-), OpAmp3.13 (IN4-), OpAmp3.2 (IN1-)
- net OpIn0: now also OpAmp1.9 (IN3-); no longer OpAmp1.10 (IN3+)
- net OpIn1: now also OpAmp1.13 (IN4-); no longer OpAmp1.12 (IN4+)
- net OpIn2: now also OpAmp1.6 (IN2-); no longer OpAmp1.5 (IN2+)
- net OpIn3: now also OpAmp1.2 (IN1-); no longer OpAmp1.3 (IN1+)
- net OpIn4: now also OpAmp2.2 (IN1-); no longer OpAmp2.3 (IN1+)
- net OpIn5: now also OpAmp2.6 (IN2-); no longer OpAmp2.5 (IN2+)
- net OpIn6: now also OpAmp2.13 (IN4-); no longer OpAmp2.12 (IN4+)
- net OpIn7: now also OpAmp2.9 (IN3-); no longer OpAmp2.10 (IN3+)
- net OpIn8: now also OpAmp3.2 (IN1-); no longer OpAmp3.3 (IN1+)
- net OpIn9: now also OpAmp3.13 (IN4-); no longer OpAmp3.12 (IN4+)
