File: PCB/main_pcb/main_pcb/main_pcb.kicad_pcb (KiCad board)
At the start: 2 copper layers, 163.5 x 133.5 mm, 56 parts, among them J1 Conn_01x20_Socket, J2 Conn_01x20_Socket, J3 Conn_01x09_Socket, Q1 DMG2305UX-7, SW0_Header1 B6B-XH-A, SW1_Header1 B6B-XH-A

Commit message: I am become death, destroyer of PCBs.
Parts:
- renumbered Photo6 to UPhoto6
Connections:
- OpAmp3 pad 10: unconnected-(OpAmp3-IN3+-Pad10) -> OpOut9
- OpAmp3 pad 5: unconnected-(OpAmp3-IN2+-Pad5) -> OpOut8
- OpAmp3 pad 6: GND -> out2
- OpAmp3 pad 7: unconnected-(OpAmp3-OUT2-Pad7) -> out2
- OpAmp3 pad 8: unconnected-(OpAmp3-OUT3-Pad8) -> out3
- OpAmp3 pad 9: GND -> out3
Routing:
- net GND: track 609.2 -> 644.0 mm
- net OpOut9: track 84.3 -> 92.2 mm
- net OpOut8: track 84.8 -> 92.6 mm
- net out2: track 0.00 -> 1.34 mm
- net out3: track 0.00 -> 1.27 mm
