File: PCB/display-pcb/display-pcb.kicad_pcb (KiCad board)
At the start: 2 copper layers, 120.5 x 57 mm, 11 parts, among them J1 B6B-XH-A, J2 B8B-XH-A, J3 B8B-XH-A, SW1 PTS645SL50-2 LFS, SW2 PTS645SL50-2 LFS, SW3 PTS645SL50-2 LFS, SW4 PTS645SL50-2 LFS, U1 NHD-C12864A1Z

Commit message: pcb finishing touches
Parts:
- added REF**: MountingHole_3.2mm_M3, MountingHole:MountingHole_3.2mm_M3, F.Cu at (237.0, 128.5)
- added REF**: MountingHole_3.2mm_M3, MountingHole:MountingHole_3.2mm_M3, F.Cu at (237.0, 67.0)
- added REF**: MountingHole_3.2mm_M3, MountingHole:MountingHole_3.2mm_M3, F.Cu at (125.0, 128.5)
- added REF**: MountingHole_3.2mm_M3, MountingHole:MountingHole_3.2mm_M3, F.Cu at (125.0, 67.0)
- J2: value B8B-XH-A -> Display_Header
- moved J3 17.5 mm to (125.5, 104.0), turned to -90 degrees
Connections:
- J2 pad 6: A0 -> /RESET
- J2 pad 7: /RESET -> A0
- J3 pad 1: SD_CSn -> SD_3V3
- J3 pad 4: SD_MISO -> GND
- J3 pad 5: GND -> SD_SCK
- J3 pad 6: SD_SCK -> SD_MISO
- J3 pad 7: GND -> SD_CSn
- J3 pad 8: SD_3V3 -> GND
Routing:
- net SD_MOSI: track 22.7 -> 25.8 mm
- net SD_SCK: track 14.5 -> 16.5 mm
- net SD_CSn: track 27.3 -> 26.2 mm
- net SD_MISO: track 19.1 -> 20.1 mm
Other:
- board size 120.5 x 57 mm -> 120.8 x 69 mm

Commit message: gerbs
Connections:
- J2 pad 6: /RESET -> A0
- J2 pad 7: A0 -> /RESET
Changed lines of the file:
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@@
 			(plot_on_all_layers_selection 0x00000000_00000000_00000000_00000000)
 			(disableapertmacros no)
-			(usegerberextensions no)
+			(usegerberextensions yes)
 			(usegerberattributes yes)
 			(usegerberadvancedattributes yes)
@@
 			(sketchdnponfab yes)
 			(crossoutdnponfab yes)
-			(subtractmaskfromsilk no)
+			(subtractmaskfromsilk yes)
 			(outputformat 1)
 			(mirror no)
 			(drillshape 0)
 			(scaleselection 1)
-			(outputdirectory "gerber/")
+			(outputdirectory "gerber_files/")
 		)
 	)
@@
 			(layers "*.Cu" "*.Mask")
 			(remove_unused_layers no)
-			(net 22 "{slash}RESET")
+			(net 19 "A0")
 			(pinfunction "6")
 			(pintype "passive")
@@
 			(layers "*.Cu" "*.Mask")
 			(remove_unused_layers no)
-			(net 19 "A0")
+			(net 22 "{slash}RESET")
 			(pinfunction "7")
 			(pintype "passive")
