File: PCB/power_splitter - NEW/power_splitter.kicad_pcb (KiCad board)
At the start: 2 copper layers, 57.1 x 48.5 mm, 36 parts, among them J1 B02P-VL, J2 B02P-VL, J3 B02P-VL, J4 PJ-082BH, J5 B02P-VL, Q2 IRLZ44N, U1 AP62300TWU, U2 AP62300TWU

Commit message: new power PCB
Parts:
- removed C10, C4: C_Small, Capacitor_SMD:C_1206_3216Metric_Pad1.33x1.80mm_HandSolder
- removed R1, R2, R5, R6: R_Small, RESISTOR:YAG_MF25_YAG
- moved U2 7.61 mm to (89.5, 58.5), turned to 90 degrees
- moved C8 3.90 mm to (118.9, 59.5), turned to 180 degrees
- moved C3 2.55 mm to (96.5, 58.5), turned to -90 degrees
- turned U1 to 90 degrees
- renumbered T_Fuse_1 to Thermal_Fuse_1, T_Fuse_2 to Thermal_Fuse_2
Connections:
- C2 pad 1: Net-(U2-EN) -> Net-(U2-BST)
- C3 pad 1: Net-(U2-BST) -> Net-(U2-IN)
- C8 pad 1: Net-(U1-BST) -> Net-(U1-IN)
- Thermal_Fuse_2 pad 2: Net-(U2-EN) -> Net-(U2-BST)
- U1 pad 3: 5V_Line -> Net-(U1-IN)
- U1 pad 4: Net-(U1-FB) -> 3V_Line
- U1 pad 5: 5V_Line -> unconnected-(U1-EN-Pad5)
- U1 pad 6: Net-(U1-BST) -> 5V_Line
- U2 pad 3: Net-(U2-EN) -> Net-(U2-IN)
- U2 pad 4: Net-(U2-FB) -> 5V_Line
- U2 pad 5: Net-(U2-EN) -> unconnected-(U2-EN-Pad5)
Routing:
- net Net-(U2-FB): track 27.1 -> 0.00 mm
- net Net-(U1-FB): track 26.1 -> 0.00 mm
- net Net-(U2-BST): track 3.69 -> 26.4 mm
- net Net-(U2-EN): track 21.0 -> 0.00 mm
- net 3V_Line: track 40.4 -> 49.5 mm
- net Net-(U1-SW): track 14.3 -> 21.8 mm
- net Net-(U1-IN): track 0.00 -> 7.50 mm
- net Net-(U2-IN): track 0.00 -> 7.17 mm
- net Net-(U2-SW): track 10.6 -> 16.4 mm
- net 5V_Line: track 64.8 -> 59.8 mm
- net GND: track 56.1 -> 51.3 mm, vias 18 -> 16
- net Net-(U1-BST): track 4.01 -> 0.00 mm
Other:
- board text added: "${REFERENCE}"
