File: PCB/power_splitter - NEW/power_splitter.kicad_sch (KiCad schematic)
At the start: 32 parts, among them J1 B02P-VL, J2 B02P-VL, J3 B02P-VL, J4 PJ-082BH, J5 B02P-VL, Q2 IRLZ44N, U1 AP62300TWU, U2 AP62300TWU

Commit message: trying again
Parts:
- removed C10, C4: C_Small, Capacitor_SMD:C_1206_3216Metric_Pad1.33x1.80mm_HandSolder, symbol Device:C_Small
- removed R1, R2, R5, R6: R_Small, RESISTOR:YAG_MF25_YAG, symbol Device:R_Small
Connections:
- net 3V_Line: now also U1.4 (FB)
- net 5V_Line: now also U1.6 (BST), U2.4 (FB); no longer U1.3 (IN), U1.5 (EN)
- net at C8.1: now also U1.3 (IN); no longer U1.6 (BST)
Other:
- note removed: "100p"
- note removed: "33.2k"
- note removed: "56.2k"
